Commit message: MAPS can now be loaded into gazebo
MAPS can now be loaded into gazebo

File: maps/maps_description/urdf/maps.xacro (robot description, xacro)
@@ -5,5 +5,5 @@
   <xacro:macro name="maps" params="name parent offset_x offset_y offset_z offset_roll offset_pitch offset_yaw">
     <link name="${name}_base_link">
-      <inertial>
+      <!-- <inertial>
         <origin xyz="0 0 0" rpy="0 0 0"/>
         <mass value="0.0"/>
@@ -20,5 +20,5 @@
         <geometry>
         </geometry>
-      </collision>
+      </collision> -->
     </link>
     <link name="${name}_bottom_plate">
@@ -31,12 +31,12 @@
         <origin xyz="0 0 0" rpy="0 0 0"/>
         <geometry>
-          <mesh filename="package://maps_description/meshes/bottom_plate.stl" scale="0.001 0.001 0.001"/>
-        </geometry>
-        <material name="black"/>
-      </visual>
-      <collision>
-        <origin xyz="0 0 0" rpy="0 0 0"/>
-        <geometry>
-          <mesh filename="package://maps_description/meshes/bottom_plate.stl" scale="0.001 0.001 0.001"/>
+          <mesh filename="file://$(find maps_description)/meshes/bottom_plate.stl" scale="0.001 0.001 0.001"/>
+        </geometry>
+        <material name="black"/>
+      </visual>
+      <collision>
+        <origin xyz="0 0 0" rpy="0 0 0"/>
+        <geometry>
+          <mesh filename="file://$(find maps_description)/meshes/bottom_plate.stl" scale="0.001 0.001 0.001"/>
         </geometry>
       </collision>
@@ -51,5 +51,5 @@
         <origin xyz="-0.0287 0.059285 -0.048891" rpy="0 0 0"/>
         <geometry>
-          <mesh filename="package://maps_description/meshes/Stepper_Housing_1.stl" scale="0.001 0.001 0.001"/>
+          <mesh filename="file://$(find maps_description)/meshes/Stepper_Housing_1.stl" scale="0.001 0.001 0.001"/>
         </geometry>
         <material name="black"/>
@@ -58,5 +58,5 @@
         <origin xyz="-0.0287 0.059285 -0.048891" rpy="0 0 0"/>
         <geometry>
-          <mesh filename="package://maps_description/meshes/Stepper_Housing_1.stl" scale="0.001 0.001 0.001"/>
+          <mesh filename="file://$(find maps_description)/meshes/Stepper_Housing_1.stl" scale="0.001 0.001 0.001"/>
         </geometry>
       </collision>
@@ -71,5 +71,5 @@
         <origin xyz="-0.049606 0.045344 -0.111388" rpy="0 0 0"/>
         <geometry>
-          <mesh filename="package://maps_description/meshes/Stepper_Motor_2.stl" scale="0.001 0.001 0.001"/>
+          <mesh filename="file://$(find maps_description)/meshes/Stepper_Motor_2.stl" scale="0.001 0.001 0.001"/>
         </geometry>
         <material name="silver"/>
@@ -78,5 +78,5 @@
         <origin xyz="-0.049606 0.045344 -0.111388" rpy="0 0 0"/>
         <geometry>
-          <mesh filename="package://maps_description/meshes/Stepper_Motor_2.stl" scale="0.001 0.001 0.001"/>
+          <mesh filename="file://$(find maps_description)/meshes/Stepper_Motor_2.stl" scale="0.001 0.001 0.001"/>
         </geometry>
       </collision>
@@ -91,5 +91,5 @@
         <origin xyz="-0.0287 -0.011715 -0.073891" rpy="0 0 0"/>
         <geometry>
-          <mesh filename="package://maps_description/meshes/Stepper_Motor_Pulley_2.stl" scale="0.001 0.001 0.001"/>
+          <mesh filename="file://$(find maps_description)/meshes/Stepper_Motor_Pulley_2.stl" scale="0.001 0.001 0.001"/>
         </geometry>
         <material name="silver"/>
@@ -98,5 +98,5 @@
         <origin xyz="-0.0287 -0.011715 -0.073891" rpy="0 0 0"/>
         <geometry>
-          <mesh filename="package://maps_description/meshes/Stepper_Motor_Pulley_2.stl" scale="0.001 0.001 0.001"/>
+          <mesh filename="file://$(find maps_description)/meshes/Stepper_Motor_Pulley_2.stl" scale="0.001 0.001 0.001"/>
         </geometry>
       </collision>
@@ -111,5 +111,5 @@
         <origin xyz="-0.049606 0.045344 -0.048888" rpy="0 0 0"/>
         <geometry>
-          <mesh filename="package://maps_description/meshes/Stepper_Motor_1.stl" scale="0.001 0.001 0.001"/>
+          <mesh filename="file://$(find maps_description)/meshes/Stepper_Motor_1.stl" scale="0.001 0.001 0.001"/>
         </geometry>
         <material name="silver"/>
@@ -118,5 +118,5 @@
         <origin xyz="-0.049606 0.045344 -0.048888" rpy="0 0 0"/>
         <geometry>
-          <mesh filename="package://maps_description/meshes/Stepper_Motor_1.stl" scale="0.001 0.001 0.001"/>
+          <mesh filename="file://$(find maps_description)/meshes/Stepper_Motor_1.stl" scale="0.001 0.001 0.001"/>
         </geometry>
       </collision>
@@ -131,5 +131,5 @@
         <origin xyz="-0.0287 -0.011715 -0.073891" rpy="0 0 0"/>
         <geometry>
-          <mesh filename="package://maps_description/meshes/Stepper_Motor_Pulley_1.stl" scale="0.001 0.001 0.001"/>
+          <mesh filename="file://$(find maps_description)/meshes/Stepper_Motor_Pulley_1.stl" scale="0.001 0.001 0.001"/>
         </geometry>
         <material name="silver"/>
@@ -138,5 +138,5 @@
         <origin xyz="-0.0287 -0.011715 -0.073891" rpy="0 0 0"/>
         <geometry>
-          <mesh filename="package://maps_description/meshes/Stepper_Motor_Pulley_1.stl" scale="0.001 0.001 0.001"/>
+          <mesh filename="file://$(find maps_description)/meshes/Stepper_Motor_Pulley_1.stl" scale="0.001 0.001 0.001"/>
         </geometry>
       </collision>
@@ -151,5 +151,5 @@
         <origin xyz="-0.054412 0.011344 -0.043888" rpy="0 0 0"/>
         <geometry>
-          <mesh filename="package://maps_description/meshes/Housing_Half_Right_1.stl" scale="0.001 0.001 0.001"/>
+          <mesh filename="file://$(find maps_description)/meshes/Housing_Half_Right_1.stl" scale="0.001 0.001 0.001"/>
         </geometry>
         <material name="black"/>
@@ -158,5 +158,5 @@
         <origin xyz="-0.054412 0.011344 -0.043888" rpy="0 0 0"/>
         <geometry>
-          <mesh filename="package://maps_description/meshes/Housing_Half_Right_1.stl" scale="0.001 0.001 0.001"/>
+          <mesh filename="file://$(find maps_description)/meshes/Housing_Half_Right_1.stl" scale="0.001 0.001 0.001"/>
         </geometry>
       </collision>
@@ -171,5 +171,5 @@
         <origin xyz="-0.053812 -0.025156 0.066112" rpy="0 0 0"/>
         <geometry>
-          <mesh filename="package://maps_description/meshes/Lid_1.stl" scale="0.001 0.001 0.001"/>
+          <mesh filename="file://$(find maps_description)/meshes/Lid_1.stl" scale="0.001 0.001 0.001"/>
         </geometry>
         <material name="black"/>
@@ -178,5 +178,5 @@
         <origin xyz="-0.053812 -0.025156 0.066112" rpy="0 0 0"/>
         <geometry>
-          <mesh filename="package://maps_description/meshes/Lid_1.stl" scale="0.001 0.001 0.001"/>
+          <mesh filename="file://$(find maps_description)/meshes/Lid_1.stl" scale="0.001 0.001 0.001"/>
         </geometry>
       </collision>
@@ -191,5 +191,5 @@
         <origin xyz="-0.014706 -0.00794 3e-06" rpy="0 0 0"/>
         <geometry>
-          <mesh filename="package://maps_description/meshes/Heat_Set_Nitinol_Tubing_1.stl" scale="0.001 0.001 0.001"/>
+          <mesh filename="file://$(find maps_description)/meshes/Heat_Set_Nitinol_Tubing_1.stl" scale="0.001 0.001 0.001"/>
         </geometry>
         <material name="silver"/>
@@ -198,5 +198,5 @@
         <origin xyz="-0.014706 -0.00794 3e-06" rpy="0 0 0"/>
         <geometry>
-          <mesh filename="package://maps_description/meshes/Heat_Set_Nitinol_Tubing_1.stl" scale="0.001 0.001 0.001"/>
+          <mesh filename="file://$(find maps_description)/meshes/Heat_Set_Nitinol_Tubing_1.stl" scale="0.001 0.001 0.001"/>
         </geometry>
       </collision>
@@ -211,5 +211,5 @@
         <origin xyz="-0.092112 -0.015881 0.071823" rpy="0 0 0"/>
         <geometry>
-          <mesh filename="package://maps_description/meshes/Clamp_1.stl" scale="0.001 0.001 0.001"/>
+          <mesh filename="file://$(find maps_description)/meshes/Clamp_1.stl" scale="0.001 0.001 0.001"/>
         </geometry>
         <material name="silver"/>
@@ -218,5 +218,5 @@
         <origin xyz="-0.092112 -0.015881 0.071823" rpy="0 0 0"/>
         <geometry>
-          <mesh filename="package://maps_description/meshes/Clamp_1.stl" scale="0.001 0.001 0.001"/>
+          <mesh filename="file://$(find maps_description)/meshes/Clamp_1.stl" scale="0.001 0.001 0.001"/>
         </geometry>
       </collision>
@@ -231,5 +231,5 @@
         <origin xyz="-0.08886 -0.011717 0.091848" rpy="0 0 0"/>
         <geometry>
-          <mesh filename="package://maps_description/meshes/9271K713_Torsion_Spring_1.stl" scale="0.001 0.001 0.001"/>
+          <mesh filename="file://$(find maps_description)/meshes/9271K713_Torsion_Spring_1.stl" scale="0.001 0.001 0.001"/>
         </geometry>
         <material name="silver"/>
@@ -238,5 +238,5 @@
         <origin xyz="-0.08886 -0.011717 0.091848" rpy="0 0 0"/>
         <geometry>
-          <mesh filename="package://maps_description/meshes/9271K713_Torsion_Spring_1.stl" scale="0.001 0.001 0.001"/>
+          <mesh filename="file://$(find maps_description)/meshes/9271K713_Torsion_Spring_1.stl" scale="0.001 0.001 0.001"/>
         </geometry>
       </collision>
@@ -251,5 +251,5 @@
         <origin xyz="-0.073212 -0.015881 0.039665" rpy="0 0 0"/>
         <geometry>
-          <mesh filename="package://maps_description/meshes/Carriage_1.stl" scale="0.001 0.001 0.001"/>
+          <mesh filename="file://$(find maps_description)/meshes/Carriage_1.stl" scale="0.001 0.001 0.001"/>
         </geometry>
         <material name="silver"/>
@@ -258,5 +258,5 @@
         <origin xyz="-0.073212 -0.015881 0.039665" rpy="0 0 0"/>
         <geometry>
-          <mesh filename="package://maps_description/meshes/Carriage_1.stl" scale="0.001 0.001 0.001"/>
+          <mesh filename="file://$(find maps_description)/meshes/Carriage_1.stl" scale="0.001 0.001 0.001"/>
         </geometry>
       </collision>
@@ -271,5 +271,5 @@
         <origin xyz="-0.073212 -0.015881 6e-06" rpy="0 0 0"/>
         <geometry>
-          <mesh filename="package://maps_description/meshes/Encoder_1.stl" scale="0.001 0.001 0.001"/>
+          <mesh filename="file://$(find maps_description)/meshes/Encoder_1.stl" scale="0.001 0.001 0.001"/>
         </geometry>
         <material name="silver"/>
@@ -278,5 +278,5 @@
         <origin xyz="-0.073212 -0.015881 6e-06" rpy="0 0 0"/>
         <geometry>
-          <mesh filename="package://maps_description/meshes/Encoder_1.stl" scale="0.001 0.001 0.001"/>
+          <mesh filename="file://$(find maps_description)/meshes/Encoder_1.stl" scale="0.001 0.001 0.001"/>
         </geometry>
       </collision>
@@ -291,5 +291,5 @@
         <origin xyz="-0.037412 -0.022156 0.068612" rpy="0 0 0"/>
         <geometry>
-          <mesh filename="package://maps_description/meshes/Housing_Half_Left_1.stl" scale="0.001 0.001 0.001"/>
+          <mesh filename="file://$(find maps_description)/meshes/Housing_Half_Left_1.stl" scale="0.001 0.001 0.001"/>
         </geometry>
         <material name="black"/>
@@ -298,5 +298,5 @@
         <origin xyz="-0.037412 -0.022156 0.068612" rpy="0 0 0"/>
         <geometry>
-          <mesh filename="package://maps_description/meshes/Housing_Half_Left_1.stl" scale="0.001 0.001 0.001"/>
+          <mesh filename="file://$(find maps_description)/meshes/Housing_Half_Left_1.stl" scale="0.001 0.001 0.001"/>
         </geometry>
       </collision>
