Commit message: Finish oct_description; @wip work on oct_gazebo; @wip start oct_plugin

File: oct/oct_description/urdf/hc_sr04.xacro (robot description, xacro)
@@ -5,5 +5,5 @@
         <origin xyz="0 0 0" rpy="1.57 0 1.57"/>
         <geometry>
-          <mesh filename="file://$(find edumip_description)/meshes/HC-SR04.stl" scale="0.001 0.001 0.001"/>
+          <mesh filename="file://$(find oct_description)/meshes/HC-SR04.stl" scale="0.001 0.001 0.001"/>
         </geometry>
         <material name="red">
@@ -15,5 +15,5 @@
         <origin xyz="0 0 0" rpy="1.57 0 1.57"/>
         <geometry>
-          <mesh filename="file://$(find edumip_description)/meshes/HC-SR04.stl" scale="0.001 0.001 0.001"/>
+          <mesh filename="file://$(find oct_description)/meshes/HC-SR04.stl" scale="0.001 0.001 0.001"/>
         </geometry>
         <material name="red">

File: oct/oct_description/urdf/oct.urdf.xacro (robot description, xacro)
@@ -1,6 +1,7 @@
 <robot xmlns:xacro="http://www.ros.org/wiki/xacro"  name="oct_test">
   <xacro:include filename="$(find oct_description)/urdf/oct.xacro" />
-  <xacro:oct_test name="oct" parent="world_link">
+  <link name="world" />
+  <xacro:oct parent="world">
     <origin xyz="0 0 0.1" rpy="0 0 0"/>
-  </xacro:oct_test>
+  </xacro:oct>
 </robot>

File: oct/oct_description/urdf/oct.xacro (robot description, xacro)
@@ -1,10 +1,10 @@
 <robot xmlns:xacro="http://www.ros.org/wiki/xacro"  name="oct">
-  <xacro:include filename="$(find edumip_description)/urdf/hc_sr04.xacro" />
+  <xacro:include filename="$(find oct_description)/urdf/hc_sr04.xacro" />
   <xacro:macro name="oct" params="parent *origin">
     <xacro:hc_sr04 name="oct_tissue" id="tissue" parent="${parent}">
-      <xacro:insert_block name="${origin}"/>
+      <xacro:insert_block name="origin"/>
     </xacro:hc_sr04>
     <xacro:hc_sr04 name="oct_nitinol" id="nitinol" parent="${parent}">
-      <xacro:insert_block name="${origin}"/>
+      <xacro:insert_block name="origin"/>
     </xacro:hc_sr04>
   </xacro:macro>

Commit message: Add minimal example for gpu_lidar and selective sensing for models in gazebo

File: oct/oct_description/urdf/hc_sr04.xacro (robot description, xacro)
@@ -11,5 +11,4 @@
         </material>
       </visual>
-      <!--
       <collision>
         <origin xyz="0 0 0" rpy="1.57 0 1.57"/>
@@ -21,5 +20,4 @@
         </material>
       </collision>
-      -->
     </link>
     <joint name="sonar_joint_${id}" type="fixed">
@@ -33,4 +31,27 @@
       </plugin>
     </gazebo>
+    <gazebo reference="sonar_link_${id}">
+      <sensor type="camera" name="${name}">
+        <camera>
+					<horizontal_fov>1.047</horizontal_fov>
+					<image>
+						<width>320</width>
+						<height>240</height>
+					</image>
+					<clip>
+						<near>0.1</near>
+						<far>100</far>
+					</clip>
+				</camera>
+        <visibility_mask>4294967294</visibility_mask>
+        <update_rate>30</update_rate>
+        <always_on>1</always_on>
+        <topic>camera</topic>
+        <visualize>1</visualize>
+        <plugin filename="ignition-gazebo-sensors-system" name="ignition::gazebo::systems::Sensors">
+        </plugin>
+      </sensor>
+    </gazebo>
+    <!--
     <gazebo reference="sonar_link_${id}">
       <sensor type="gpu_lidar" name="${name}">
@@ -64,4 +85,5 @@
       </sensor>
     </gazebo>
+    -->
   </xacro:macro>
 </robot>

File: oct/oct_description/urdf/oct.urdf.xacro (robot description, xacro)
@@ -1,5 +1,26 @@
-<robot xmlns:xacro="http://www.ros.org/wiki/xacro"  name="oct_test">
+<robot xmlns:xacro="http://www.ros.org/wiki/xacro"  name="oct">
   <xacro:include filename="$(find oct_description)/urdf/oct.xacro" />
-  <link name="world" />
+  <link name="world">
+    <visual>
+      <origin rpy="0 -0.20 0" xyz="0 0 0.05"/>
+      <geometry>
+        <box size="0.035 0.05 0.1"/>
+      </geometry>
+      <material name="Blue">
+        <color rgba="0 0.0 1.0 0.5"/>
+      </material>
+    </visual>
+    <collision>
+      <origin rpy="0 -0.20 0" xyz="0 0 0.05"/>
+      <geometry>
+        <box size="0.035 0.05 0.1"/>
+      </geometry>
+    </collision>
+    <inertial>
+      <origin rpy="0 0 0" xyz="0 0 0.05"/>
+      <mass value="0.180"/>
+      <inertia ixx="6.0e-4" ixy="0" ixz="0" iyy="6.0e-4" iyz="0" izz="6.0e-4"/>
+    </inertial>
+  </link>
   <xacro:oct parent="world">
     <origin xyz="0 0 0.1" rpy="0 0 0"/>

File: oct/oct_description/urdf/oct.xacro (robot description, xacro)
@@ -2,4 +2,32 @@
   <xacro:include filename="$(find oct_description)/urdf/hc_sr04.xacro" />
   <xacro:macro name="oct" params="parent *origin">
+    <link name="base_link">
+      <visual>
+        <origin rpy="0 -0.20 0" xyz="0 0 0.05"/>
+        <geometry>
+          <box size="0.035 0.05 0.1"/>
+        </geometry>
+        <material name="Blue">
+          <color rgba="0 0.0 1.0 0.5"/>
+        </material>
+      </visual>
+      <collision>
+        <origin rpy="0 -0.20 0" xyz="0 0 0.05"/>
+        <geometry>
+          <box size="0.035 0.05 0.1"/>
+        </geometry>
+      </collision>
+      <inertial>
+        <origin rpy="0 0 0" xyz="0 0 0.05"/>
+        <mass value="0.180"/>
+        <inertia ixx="6.0e-4" ixy="0" ixz="0" iyy="6.0e-4" iyz="0" izz="6.0e-4"/>
+      </inertial>
+    </link>
+    <joint name="base_link_joint" type="fixed">
+      <parent link="${parent}"/>
+      <child link="base_link"/>
+      <xacro:insert_block name="origin"/>
+      <axis xyz="0 1 0"/>
+    </joint>
     <xacro:hc_sr04 name="oct_tissue" id="tissue" parent="${parent}">
       <xacro:insert_block name="origin"/>
