Commit message: Finish first cut of oct_gazebo with working example

File: oct/oct_description/urdf/oct.xacro (robot description, xacro)
@@ -40,13 +40,13 @@
       <parent link="oct_link"/>
       <child link="oct_tissue_link"/>
-      <origin xyz="0 0 0"/>
+      <origin xyz="0 0 0" rpy="0 1.57 0"/><!-- orient lidar along model; it naturally points in x-direction -->
     </joint>
     <joint name="oct_nitinol_joint" type="fixed">
       <parent link="oct_link"/>
       <child link="oct_nitinol_link"/>
-      <origin xyz="0 0 0"/>
+      <origin xyz="0 0 0" rpy="0 1.57 0"/>
     </joint>
     <gazebo reference="oct_tissue_link">
-      <sensor type="gpu_lidar" name="gpu_lidar">
+      <sensor type="gpu_lidar" name="oct_tissue_lidar">
         <update_rate>40.0</update_rate>
         <always_on>1</always_on>
@@ -75,10 +75,12 @@
           <visibility_mask>${tissue_visibility_mask}</visibility_mask>
         </ray>
+        <!--
         <plugin filename="ignition-gazebo-sensors-system" name="ignition::gazebo::systems::Sensors">
         </plugin>
+        -->
       </sensor>
     </gazebo>
     <gazebo reference="oct_nitinol_link">
-      <sensor type="gpu_lidar" name="gpu_lidar">
+      <sensor type="gpu_lidar" name="oct_nitinol_lidar">
         <update_rate>40.0</update_rate>
         <always_on>1</always_on>
@@ -107,6 +109,8 @@
           <visibility_mask>${nitinol_visibility_mask}</visibility_mask>
         </ray>
+        <!--
         <plugin filename="ignition-gazebo-sensors-system" name="ignition::gazebo::systems::Sensors">
         </plugin>
+        -->
       </sensor>
     </gazebo>
