Commit message: @wip begin setting up new mesh and xacro for oct

File: oct/oct_description/urdf/oct.urdf.xacro (robot description, xacro)
@@ -1,26 +1,4 @@
 <robot xmlns:xacro="http://www.ros.org/wiki/xacro"  name="oct">
   <xacro:include filename="$(find oct_description)/urdf/oct.xacro" />
-  <link name="world">
-    <visual>
-      <origin rpy="0 -0.20 0" xyz="0 0 0.05"/>
-      <geometry>
-        <box size="0.035 0.05 0.1"/>
-      </geometry>
-      <material name="Blue">
-        <color rgba="0 0.0 1.0 0.5"/>
-      </material>
-    </visual>
-    <collision>
-      <origin rpy="0 -0.20 0" xyz="0 0 0.05"/>
-      <geometry>
-        <box size="0.035 0.05 0.1"/>
-      </geometry>
-    </collision>
-    <inertial>
-      <origin rpy="0 0 0" xyz="0 0 0.05"/>
-      <mass value="0.180"/>
-      <inertia ixx="6.0e-4" ixy="0" ixz="0" iyy="6.0e-4" iyz="0" izz="6.0e-4"/>
-    </inertial>
-  </link>
   <xacro:oct parent="world">
     <origin xyz="0 0 0.1" rpy="0 0 0"/>

File: oct/oct_description/urdf/oct.xacro (robot description, xacro)
@@ -1,39 +1,43 @@
 <robot xmlns:xacro="http://www.ros.org/wiki/xacro"  name="oct">
-  <xacro:include filename="$(find oct_description)/urdf/hc_sr04.xacro" />
   <xacro:macro name="oct" params="parent *origin">
-    <link name="base_link">
+    <link name="oct_link">
       <visual>
-        <origin rpy="0 -0.20 0" xyz="0 0 0.05"/>
+        <xacro:insert_block name="origin"/>
         <geometry>
-          <box size="0.035 0.05 0.1"/>
+          <cylinder length="0.01" radius="0.001"/>
         </geometry>
-        <material name="Blue">
-          <color rgba="0 0.0 1.0 0.5"/>
+        <material name="blue">
+          <color rgba="0.0 0.0 0.8 1.0"/>
         </material>
       </visual>
       <collision>
-        <origin rpy="0 -0.20 0" xyz="0 0 0.05"/>
+        <origin xyz="0 0 0"/>
         <geometry>
-          <box size="0.035 0.05 0.1"/>
+          <cylinder length="0.01" radius="0.001"/>
         </geometry>
+        <material name="blue">
+          <color rgba="0.0 0.0 0.8 1.0"/>
+        </material>
       </collision>
       <inertial>
-        <origin rpy="0 0 0" xyz="0 0 0.05"/>
-        <mass value="0.180"/>
+        <origin rpy="0 0 0" xyz="0 0 0"/>
+        <mass value="0.000453592"/>
         <inertia ixx="6.0e-4" ixy="0" ixz="0" iyy="6.0e-4" iyz="0" izz="6.0e-4"/>
       </inertial>
     </link>
-    <joint name="base_link_joint" type="fixed">
-      <parent link="${parent}"/>
-      <child link="base_link"/>
-      <xacro:insert_block name="origin"/>
+    <link name="oct_tissue_link"/>
+    <link name="oct_nitinol_link"/>
+    <joint name="oct_tissue_joint" type="fixed">
+      <parent link="oct_link"/>
+      <child link="oct_tissue_link"/>
+      <origin xyz="0 0 0"/>
       <axis xyz="0 1 0"/>
     </joint>
-    <xacro:hc_sr04 name="oct_tissue" id="tissue" parent="${parent}">
-      <xacro:insert_block name="origin"/>
-    </xacro:hc_sr04>
-    <xacro:hc_sr04 name="oct_nitinol" id="nitinol" parent="${parent}">
-      <xacro:insert_block name="origin"/>
-    </xacro:hc_sr04>
+    <joint name="oct_nitinol_joint" type="fixed">
+      <parent link="oct_link"/>
+      <child link="oct_nitinol_link"/>
+      <origin xyz="0 0 0"/>
+      <axis xyz="0 1 0"/>
+    </joint>
   </xacro:macro>
 </robot>

Commit message: Rebuild oct model and launch

File: oct/oct_description/urdf/oct.urdf.xacro (robot description, xacro)
@@ -1,6 +1,13 @@
 <robot xmlns:xacro="http://www.ros.org/wiki/xacro"  name="oct">
   <xacro:include filename="$(find oct_description)/urdf/oct.xacro" />
-  <xacro:oct parent="world">
-    <origin xyz="0 0 0.1" rpy="0 0 0"/>
+  <xacro:arg name="parent" default="world"/>
+  <xacro:arg name="offset_x" default="0"/>
+  <xacro:arg name="offset_y" default="0"/>
+  <xacro:arg name="offset_z" default="0"/>
+  <xacro:arg name="offset_roll" default="0"/>
+  <xacro:arg name="offset_pitch" default="0"/>
+  <xacro:arg name="offset_yaw" default="0"/>
+  <xacro:oct parent="$(arg parent)">
+		<origin xyz="$(arg offset_x) $(arg offset_y) $(arg offset_z)" rpy="$(arg offset_roll) $(arg offset_pitch) $(arg offset_yaw)"/>
   </xacro:oct>
 </robot>

File: oct/oct_description/urdf/oct.xacro (robot description, xacro)
@@ -32,5 +32,4 @@
       <child link="oct_tissue_link"/>
       <origin xyz="0 0 0"/>
-      <axis xyz="0 1 0"/>
     </joint>
     <joint name="oct_nitinol_joint" type="fixed">
@@ -38,5 +37,4 @@
       <child link="oct_nitinol_link"/>
       <origin xyz="0 0 0"/>
-      <axis xyz="0 1 0"/>
     </joint>
   </xacro:macro>

Commit message: Finish first cut of oct_description

File: oct/oct_description/urdf/oct.urdf.xacro (robot description, xacro)
@@ -8,5 +8,7 @@
   <xacro:arg name="offset_pitch" default="0"/>
   <xacro:arg name="offset_yaw" default="0"/>
-  <xacro:oct parent="$(arg parent)">
+  <xacro:arg name="tissue_visibility_mask" default="4294967294"/>
+  <xacro:arg name="nitinol_visibility_mask" default="4294967293"/>
+  <xacro:oct parent="$(arg parent)" tissue_visibility_mask="$(arg tissue_visibility_mask)" nitinol_visibility_mask="$(arg nitinol_visibility_mask)">
 		<origin xyz="$(arg offset_x) $(arg offset_y) $(arg offset_z)" rpy="$(arg offset_roll) $(arg offset_pitch) $(arg offset_yaw)"/>
   </xacro:oct>

File: oct/oct_description/urdf/oct.xacro (robot description, xacro)
@@ -1,7 +1,9 @@
 <robot xmlns:xacro="http://www.ros.org/wiki/xacro"  name="oct">
-  <xacro:macro name="oct" params="parent *origin">
+  <xacro:macro name="oct" params="parent tissue_visibility_mask nitinol_visibility_mask *origin ">
+    <!-- test code -->
+    <link name="world"/>
+    <!---->
     <link name="oct_link">
       <visual>
-        <xacro:insert_block name="origin"/>
         <geometry>
           <cylinder length="0.01" radius="0.001"/>
@@ -26,6 +28,13 @@
       </inertial>
     </link>
-    <link name="oct_tissue_link"/>
-    <link name="oct_nitinol_link"/>
+    <link name="oct_tissue_link">
+    </link>
+    <link name="oct_nitinol_link">
+    </link>
+    <joint name="oct_joint" type="fixed">
+      <parent link="${parent}"/>
+      <child link="oct_link"/>
+      <xacro:insert_block name="origin"/>
+    </joint>
     <joint name="oct_tissue_joint" type="fixed">
       <parent link="oct_link"/>
@@ -38,4 +47,68 @@
       <origin xyz="0 0 0"/>
     </joint>
+    <gazebo reference="oct_tissue_link">
+      <sensor type="gpu_lidar" name="gpu_lidar">
+        <update_rate>40.0</update_rate>
+        <always_on>1</always_on>
+        <topic>oct_tissue</topic>
+        <visualize>1</visualize>
+        <ignition_frame_id>oct_tissue_link</ignition_frame_id>
+        <ray>
+          <scan>
+            <horizontal>
+              <samples>15</samples>
+              <resolution>1.0</resolution>
+              <min_angle>-0.1309</min_angle>
+              <max_angle>0.1309</max_angle>
+            </horizontal>
+            <vertical>
+              <samples>15</samples>
+              <resolution>1.0</resolution>
+              <min_angle>-0.1309</min_angle>
+              <max_angle>0.1309</max_angle>
+            </vertical>
+          </scan>
+          <range>
+            <min>0.000001</min>
+            <max>4.0</max>
+          </range>
+          <visibility_mask>${tissue_visibility_mask}</visibility_mask>
+        </ray>
+        <plugin filename="ignition-gazebo-sensors-system" name="ignition::gazebo::systems::Sensors">
+        </plugin>
+      </sensor>
+    </gazebo>
+    <gazebo reference="oct_nitinol_link">
+      <sensor type="gpu_lidar" name="gpu_lidar">
+        <update_rate>40.0</update_rate>
+        <always_on>1</always_on>
+        <topic>oct_nitinol</topic>
+        <visualize>1</visualize>
+        <ignition_frame_id>oct_nitinol_link</ignition_frame_id>
+        <ray>
+          <scan>
+            <horizontal>
+              <samples>15</samples>
+              <resolution>1.0</resolution>
+              <min_angle>-0.1309</min_angle>
+              <max_angle>0.1309</max_angle>
+            </horizontal>
+            <vertical>
+              <samples>15</samples>
+              <resolution>1.0</resolution>
+              <min_angle>-0.1309</min_angle>
+              <max_angle>0.1309</max_angle>
+            </vertical>
+          </scan>
+          <range>
+            <min>0.000001</min>
+            <max>4.0</max>
+          </range>
+          <visibility_mask>${nitinol_visibility_mask}</visibility_mask>
+        </ray>
+        <plugin filename="ignition-gazebo-sensors-system" name="ignition::gazebo::systems::Sensors">
+        </plugin>
+      </sensor>
+    </gazebo>
   </xacro:macro>
 </robot>

Commit message: Get oct_gazebo running on its own again

File: oct/oct_description/urdf/oct.urdf.xacro (robot description, xacro)
@@ -10,4 +10,5 @@
   <xacro:arg name="tissue_visibility_mask" default="4294967294"/>
   <xacro:arg name="nitinol_visibility_mask" default="4294967293"/>
+  <link name="world"/>
   <xacro:oct parent="$(arg parent)" tissue_visibility_mask="$(arg tissue_visibility_mask)" nitinol_visibility_mask="$(arg nitinol_visibility_mask)">
 		<origin xyz="$(arg offset_x) $(arg offset_y) $(arg offset_z)" rpy="$(arg offset_roll) $(arg offset_pitch) $(arg offset_yaw)"/>

File: oct/oct_description/urdf/oct.xacro (robot description, xacro)
@@ -1,8 +1,4 @@
 <robot xmlns:xacro="http://www.ros.org/wiki/xacro"  name="oct">
   <xacro:macro name="oct" params="parent tissue_visibility_mask nitinol_visibility_mask *origin ">
-    <!-- test code
-    <link name="world"/>
-    -->
-    <!---->
     <link name="oct_link">
       <visual>
