Commit message: Integrate Kuka, Suture Tool and OCT with simple example in Gazebo; Add first cut of documentation for Robot package

File: robot/urdf/robot.xacro (robot description, xacro)
@@ -1,7 +1,6 @@
 <robot xmlns:xacro="http://www.ros.org/wiki/xacro"  name="oct">
   <xacro:macro name="oct" params="parent tissue_visibility_mask nitinol_visibility_mask *origin ">
-    <!-- test code
+    <!-- test code -->
     <link name="world"/>
-    -->
     <!---->
     <link name="oct_link">

File: suture-tool/suture_tool_description/urdf/endo360.urdf (robot description, URDF)
Before this commit: robot robot, 4 links, 3 joints
Links:
- removed link endo360_base
- link endo360_link_0: geometry collision mesh filename=file:///home/nightrider/Documents/JHU/rsp/rsp_fp_ws/install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; visual mesh filename=file:///home/nightrider/Documents/JHU/rsp/rsp_fp_ws/install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
- link endo360_link_1: geometry collision mesh filename=file:///home/nightrider/Documents/JHU/rsp/rsp_fp_ws/install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; visual mesh filename=file:///home/nightrider/Documents/JHU/rsp/rsp_fp_ws/install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
- link endo360_needle: mass None -> 1e-5; geometry collision mesh filename=file:///home/nightrider/Documents/JHU/rsp/rsp_fp_ws/install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 scale=0.001 0.001 0.001; visual mesh filename=file:///home/nightrider/Documents/JHU/rsp/rsp_fp_ws/install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 scale=0.001 0.001 0.001
Joints:
- removed joint iiwa_endo360_joint
- added joint world_endo360_joint: type fixed, parent world, child endo360_link_0, origin xyz=0 0 0 rpy=0 0 0
