Commit message: @wip debug suture tool on its own

File: suture-tool/suture_tool_description/urdf/endo360.urdf.xacro (robot description, xacro)
@@ -2,4 +2,5 @@
   <xacro:arg name="parent" default="world"/>
   <xacro:include filename="$(find suture_tool_description)/urdf/endo360.xacro"/>
+  <link name="$(arg parent)"/>
   <xacro:suture_tool parent="$(arg parent)" tool_name="endo360"/>
 </robot>
