Commit message: Update README

File: suture-tool/suture_tool_description/urdf/endo360.urdf (robot description, URDF)
Before this commit: robot robot, 3 links, 3 joints
Links:
- added link world
- link endo360_link_0: geometry collision mesh filename=file:///home/nightrider/Documents/JHU/rsp/rsp_clean_ws/inst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; visual mesh filename=file:///home/nightrider/Documents/JHU/rsp/rsp_clean_ws/inst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
- link endo360_link_1: geometry collision mesh filename=file:///home/nightrider/Documents/JHU/rsp/rsp_clean_ws/inst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; visual mesh filename=file:///home/nightrider/Documents/JHU/rsp/rsp_clean_ws/inst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
- link endo360_needle: geometry collision mesh filename=file:///home/nightrider/Documents/JHU/rsp/rsp_clean_ws/inst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 scale=0.001 0.001 0.001; visual mesh filename=file:///home/nightrider/Documents/JHU/rsp/rsp_clean_ws/inst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 scale=0.001 0.001 0.001
